Commit message: merge

File: turtlebot3_description/gazebo/burger.gazebo.xacro (robot description, xacro)
@@ -3,5 +3,12 @@
   <xacro:macro name="burger_gazebo" params="prefix">
   <xacro:property name="laser_visual"  value="true"/>
-  <xacro:property name="imu_visual"    value="true"/>
+  <xacro:property name="imu_ang_vel_noise_mean" value="0.0" />
+  <xacro:property name="imu_ang_vel_noise_stddev" value="2e-4" />
+  <xacro:property name="imu_ang_vel_noise_bias_mean" value="0.0000075" />
+  <xacro:property name="imu_ang_vel_noise_bias_stddev" value="0.0000008" />
+  <xacro:property name="imu_lin_acc_noise_mean" value="0.0" />
+  <xacro:property name="imu_lin_acc_noise_stddev" value="1.7e-2" />
+  <xacro:property name="imu_lin_acc_noise_bias_mean" value="0.1" />
+  <xacro:property name="imu_lin_acc_noise_bias_stddev" value="0.001" />
   <gazebo reference="${prefix}base_link">
     <material>Gazebo/DarkGrey</material>
@@ -41,5 +48,58 @@
       <always_on>true</always_on>
       <update_rate>100.0</update_rate>
-      <visualize>${imu_visual}</visualize>
+      <imu>
+        <angular_velocity>
+          <x>
+            <noise type="gaussian">
+              <mean>${imu_ang_vel_noise_mean}</mean>
+              <stddev>${imu_ang_vel_noise_stddev}</stddev>
+              <bias_mean>${imu_ang_vel_noise_bias_mean}</bias_mean>
+              <bias_stddev>${imu_ang_vel_noise_bias_stddev}</bias_stddev>
+            </noise>
+          </x>
+          <y>
+            <noise type="gaussian">
+              <mean>${imu_ang_vel_noise_mean}</mean>
+              <stddev>${imu_ang_vel_noise_stddev}</stddev>
+              <bias_mean>${imu_ang_vel_noise_bias_mean}</bias_mean>
+              <bias_stddev>${imu_ang_vel_noise_bias_stddev}</bias_stddev>
+            </noise>
+          </y>
+          <z>
+            <noise type="gaussian">
+              <mean>${imu_ang_vel_noise_mean}</mean>
+              <stddev>${imu_ang_vel_noise_stddev}</stddev>
+              <bias_mean>${imu_ang_vel_noise_bias_mean}</bias_mean>
+              <bias_stddev>${imu_ang_vel_noise_bias_stddev}</bias_stddev>
+            </noise>
+          </z>
+        </angular_velocity>
+        <linear_acceleration>
+          <x>
+            <noise type="gaussian">
+              <mean>${imu_lin_acc_noise_mean}</mean>
+              <stddev>${imu_lin_acc_noise_stddev}</stddev>
+              <bias_mean>${imu_lin_acc_noise_bias_mean}</bias_mean>
+              <bias_stddev>${imu_lin_acc_noise_bias_stddev}</bias_stddev>
+            </noise>
+          </x>
+          <y>
+            <noise type="gaussian">
+              <mean>${imu_lin_acc_noise_mean}</mean>
+              <stddev>${imu_lin_acc_noise_stddev}</stddev>
+              <bias_mean>${imu_lin_acc_noise_bias_mean}</bias_mean>
+              <bias_stddev>${imu_lin_acc_noise_bias_stddev}</bias_stddev>
+            </noise>
+          </y>
+          <z>
+            <noise type="gaussian">
+              <mean>${imu_lin_acc_noise_mean}</mean>
+              <stddev>${imu_lin_acc_noise_stddev}</stddev>
+              <bias_mean>${imu_lin_acc_noise_bias_mean}</bias_mean>
+              <bias_stddev>${imu_lin_acc_noise_bias_stddev}</bias_stddev>
+            </noise>
+          </z>
+        </linear_acceleration>
+      </imu>
     </sensor>
   </gazebo>
@@ -67,5 +127,5 @@
     <plugin name="gazebo_ros_p3d" filename="libgazebo_ros_p3d.so">
         <ros>
-          <namespace></namespace>
+          <namespace>/</namespace>
           <remapping>odom:=ground_truth</remapping>
         </ros>
